Commit message: Updated URDF
Changed into URDF of KBot V2

File: public/cad/gpr-20241204.urdf (robot description, URDF)
Before this commit: robot gpr-20241204, 22 links, 21 joints
Links:
- removed link arm1_top
- removed link arm1_top_2
- removed link arm2_shell
- removed link arm2_shell_2
- removed link arm3_shell
- removed link arm3_shell2
- removed link body1-part
- removed link foot1
- removed link foot3
- removed link hand_shell
- removed link hand_shell_2
- removed link leg0_shell
- removed link leg0_shell_2
- removed link leg1_shell
- removed link leg1_shell3
- removed link leg2_shell
- removed link leg2_shell_2
- removed link leg3_shell2
- removed link leg3_shell22
- removed link shoulder
- removed link shoulder_2
- added link KB-B-102B_TORSO_BOTTOM, mass 15.456196869999996; collision mesh filename=meshes/KB-B-102B_TORSO_BOTTOM.stl; visual mesh filename=meshes/KB-B-102B_TORSO_BOTTOM.stl
- added link KB-C-101L_ShldYokeROLL, mass 0.5450985750000001; collision mesh filename=meshes/KB-C-101L_ShldYokeROLL.stl; visual mesh filename=meshes/KB-C-101L_ShldYokeROLL.stl
- added link KB-C-101R_R_Shoulder_Drive, mass 0.5450769340000001; collision mesh filename=meshes/KB-C-101R_R_Shoulder_Drive.stl; visual mesh filename=meshes/KB-C-101R_R_Shoulder_Drive.stl
- added link KB-C-501X_Bayonet_Adapter_Hard_Stop, mass 0.571798567; collision mesh filename=meshes/KB-C-501X_Bayonet_Adapter_Hard_Stop.stl; visual mesh filename=meshes/KB-C-501X_Bayonet_Adapter_Hard_Stop.stl
- added link KB-C-501X_Bayonet_Adapter_Hard_Stop_2, mass 0.571798567; collision mesh filename=meshes/KB-C-501X_Bayonet_Adapter_Hard_Stop_2.stl; visual mesh filename=meshes/KB-C-501X_Bayonet_Adapter_Hard_Stop_2.stl
- added link KB-D-102L_L_Hip_Yoke_Drive, mass 0.710534346; collision mesh filename=meshes/KB-D-102L_L_Hip_Yoke_Drive.stl; visual mesh filename=meshes/KB-D-102L_L_Hip_Yoke_Drive.stl
- added link KB-D-102R_R_Hip_Yoke_Drive, mass 0.7105343159999999; collision mesh filename=meshes/KB-D-102R_R_Hip_Yoke_Drive.stl; visual mesh filename=meshes/KB-D-102R_R_Hip_Yoke_Drive.stl
- added link KB-D-301L_L_Femur_Lower_Drive, mass 2.5567669129999997; collision mesh filename=meshes/KB-D-301L_L_Femur_Lower_Drive.stl; visual mesh filename=meshes/KB-D-301L_L_Femur_Lower_Drive.stl
- added link KB-D-301R_R_Femur_Lower_Drive, mass 2.556833893; collision mesh filename=meshes/KB-D-301R_R_Femur_Lower_Drive.stl; visual mesh filename=meshes/KB-D-301R_R_Femur_Lower_Drive.stl
- added link KB-D-401L_L_Shin_Drive, mass 2.062098443; collision mesh filename=meshes/KB-D-401L_L_Shin_Drive.stl; visual mesh filename=meshes/KB-D-401L_L_Shin_Drive.stl
- added link KB-D-401R_R_Shin_Drive, mass 2.0622413400000004; collision mesh filename=meshes/KB-D-401R_R_Shin_Drive.stl; visual mesh filename=meshes/KB-D-401R_R_Shin_Drive.stl
- added link KB-D-501L_L_LEG-FOOT, mass 0.49274759; collision mesh filename=meshes/KB-D-501L_L_LEG-FOOT.stl; visual mesh filename=meshes/KB-D-501L_L_LEG-FOOT.stl
- added link KB-D-501R_R_LEG-FOOT, mass 0.49274711000000004; collision mesh filename=meshes/KB-D-501R_R_LEG-FOOT.stl; visual mesh filename=meshes/KB-D-501R_R_LEG-FOOT.stl
- added link L_Bicep_Lower_Drive, mass 0.86429688; collision mesh filename=meshes/L_Bicep_Lower_Drive.stl; visual mesh filename=meshes/L_Bicep_Lower_Drive.stl
- added link L_Forearm_Upper_Drive, mass 0.67693693; collision mesh filename=meshes/L_Forearm_Upper_Drive.stl; visual mesh filename=meshes/L_Forearm_Upper_Drive.stl
- added link RS03, mass 2.5903163030000003; collision mesh filename=meshes/RS03.stl; visual mesh filename=meshes/RS03.stl
- added link RS03_2, mass 2.590428564; collision mesh filename=meshes/RS03_2.stl; visual mesh filename=meshes/RS03_2.stl
- added link RS03_3, mass 1.861434012; collision mesh filename=meshes/RS03_3.stl; visual mesh filename=meshes/RS03_3.stl
- added link RS03_4, mass 1.86146043; collision mesh filename=meshes/RS03_4.stl; visual mesh filename=meshes/RS03_4.stl
- added link R_Bicep_Lower_Drive, mass 0.8639227300000001; collision mesh filename=meshes/R_Bicep_Lower_Drive.stl; visual mesh filename=meshes/R_Bicep_Lower_Drive.stl
- added link R_Forearm_Upper_Structural, mass 0.67694019; collision mesh filename=meshes/R_Forearm_Upper_Structural.stl; visual mesh filename=meshes/R_Forearm_Upper_Structural.stl
Joints:
- removed joint L_ankle
- removed joint L_elbow
- removed joint L_hip_x
- removed joint L_hip_y
- removed joint L_hip_z
- removed joint L_knee
- removed joint L_shoulder_x
- removed joint L_shoulder_y
- removed joint L_shoulder_z
- removed joint L_wrist
- removed joint R_ankle
- removed joint R_elbow
- removed joint R_hip_x
- removed joint R_hip_y
- removed joint R_hip_z
- removed joint R_knee
- removed joint R_shoulder_x
- removed joint R_shoulder_y
- removed joint R_shoulder_z
- removed joint R_wrist
- added joint left_ankle_02: type revolute, parent KB-D-401R_R_Shin_Drive, child KB-D-501R_R_LEG-FOOT, origin xyz=-0.0313 0.2925 0.005 rpy=3.1415927 0 0, axis 0 0 1, limit lower=-0.29670597 upper=0.78539816 effort=80 velocity=5
- added joint left_elbow_02: type revolute, parent R_Bicep_Lower_Drive, child R_Forearm_Upper_Structural, origin xyz=0.01749999579319584 -0.010000000468910617 -0.13699999843121974 rpy=-1.5707963646886025 2.6794895413573272e-08 1.5707962999999985, axis 0 0 1, limit lower=0 upper=2.5307274 effort=80 velocity=5
- added joint left_hip_pitch_04: type revolute, parent KB-B-102B_TORSO_BOTTOM, child KB-D-102L_L_Hip_Yoke_Drive, origin xyz=-0.047048021999999995 -0.000737257000000005 -0.07299347924500096 rpy=-1.5707963 2.6794896523796297e-08 -1.5707963267948961, axis 0 0 1, limit lower=-1.5707963 upper=1.9198622 effort=80 velocity=5
- added joint left_hip_roll_03: type revolute, parent KB-D-102L_L_Hip_Yoke_Drive, child RS03_2, origin xyz=-0.02925 0.03 -0.071 rpy=3.1415927 1.5707963 0, axis 0 0 1, limit lower=-0.20943951 upper=2.6179939 effort=80 velocity=5
- added joint left_hip_yaw_03: type revolute, parent RS03_2, child KB-D-301R_R_Femur_Lower_Drive, origin xyz=0.0 -0.14175000000000001 -0.029799999999999997 rpy=-1.5707963071795865 0.0 0.0, axis 0 0 1, limit lower=-1.5707963 upper=1.9198622 effort=80 velocity=5
- added joint left_knee_04: type revolute, parent KB-D-301R_R_Femur_Lower_Drive, child KB-D-401R_R_Shin_Drive, origin xyz=0.019600006618339327 0.02099999745046268 -0.2119999988276073 rpy=-1.5707963646886016 2.6794893859261038e-08 1.5707962535897926, axis 0 0 1, limit lower=-2.6703538 upper=0 effort=80 velocity=5
- added joint left_shoulder_pitch_03: type revolute, parent KB-B-102B_TORSO_BOTTOM, child KB-C-101R_R_Shoulder_Drive, origin xyz=0.1249499752752948 -0.000737260654998772 0.3375065237953634 rpy=1.570796364688602 -7.320510020392135e-08 -1.5707964000000025, axis 0 0 1, limit lower=-1.9198622 upper=3.4906585 effort=80 velocity=5
- added joint left_shoulder_roll_03: type revolute, parent KB-C-101R_R_Shoulder_Drive, child RS03_3, origin xyz=-0.02525 0 -0.075 rpy=0 -1.5707963 0, axis 0 0 1, limit lower=-1.4835299 upper=0.48869219 effort=80 velocity=5
- added joint left_shoulder_yaw_02: type revolute, parent RS03_3, child R_Bicep_Lower_Drive, origin xyz=-0.013 -0.14099999871210736 -0.03025020663762125 rpy=-1.570796207179587 0.0 0.0, axis 0 0 1, limit lower=-1.7453293 upper=1.7453293 effort=80 velocity=5
- added joint left_wrist_02: type revolute, parent R_Forearm_Upper_Structural, child KB-C-501X_Bayonet_Adapter_Hard_Stop, origin xyz=0.017350000026794897 0.1055 0.018 rpy=1.5707963999999996 1.5707963000000005 0.0, axis 0 0 1, limit lower=-1.7453293 upper=1.7453293 effort=80 velocity=5
- added joint right_ankle_02: type revolute, parent KB-D-401L_L_Shin_Drive, child KB-D-501L_L_LEG-FOOT, origin xyz=-0.0313 -0.2925 0.005 rpy=0 0 0, axis 0 0 -1, limit lower=-0.29670597 upper=0.78539816 effort=80 velocity=5
- added joint right_elbow_02: type revolute, parent L_Bicep_Lower_Drive, child L_Forearm_Upper_Drive, origin xyz=-0.017499996329093773 -0.009999999531089408 -0.1370000008185232 rpy=1.5707962889011908 2.6794895413573272e-08 1.5707962999999994, axis 0 0 1, limit lower=-2.5307274 upper=0 effort=80 velocity=5
- added joint right_hip_pitch_04: type revolute, parent KB-B-102B_TORSO_BOTTOM, child KB-D-102R_R_Hip_Yoke_Drive, origin xyz=0.04704799199999996 -0.0007372588099980745 -0.07299347715499904 rpy=1.570796353589793 2.6794898300153136e-08 -1.570796373205102, axis 0 0 1, limit lower=-1.9198622 upper=1.5707963 effort=80 velocity=5
- added joint right_hip_roll_03: type revolute, parent KB-D-102R_R_Hip_Yoke_Drive, child RS03, origin xyz=-0.02925 -0.03 -0.071 rpy=0 -1.5707963 0, axis 0 0 1, limit lower=-2.6179939 upper=0.20943951 effort=80 velocity=5
- added joint right_hip_yaw_03: type revolute, parent RS03, child KB-D-301L_L_Femur_Lower_Drive, origin xyz=0.0 -0.14175 -0.029799999999999997 rpy=-1.5707963071795865 0.0 0.0, axis 0 0 1, limit lower=-1.5707963 upper=1.9198622 effort=80 velocity=5
- added joint right_knee_04: type revolute, parent KB-D-301L_L_Femur_Lower_Drive, child KB-D-401L_L_Shin_Drive, origin xyz=-0.019600005492953775 0.02099999892954119 -0.21199999882760728 rpy=1.5707963646886023 -2.6794896967885506e-08 1.5707963464102066, axis 0 0 1, limit lower=0 upper=2.6703538 effort=80 velocity=5
- added joint right_shoulder_pitch_03: type revolute, parent KB-B-102B_TORSO_BOTTOM, child KB-C-101L_ShldYokeROLL, origin xyz=-0.12495002472470498 -0.0007372555262804718 0.33750651980463664 rpy=-1.5707963182783953 2.6794895635617877e-08 1.5707962999999996, axis 0 0 -1, limit lower=-1.9198622 upper=3.4906585 effort=80 velocity=5
- added joint right_shoulder_roll_03: type revolute, parent KB-C-101L_ShldYokeROLL, child RS03_4, origin xyz=0.02525 0 0.075 rpy=3.1415927 -1.5707963 0, axis 0 0 1, limit lower=-0.48869219 upper=1.4835299 effort=80 velocity=5
- added joint right_shoulder_yaw_02: type revolute, parent RS03_4, child L_Bicep_Lower_Drive, origin xyz=0.012999999999999998 -0.14099999871210692 -0.03025021299389611 rpy=-1.5707962143591734 0.0 0.0, axis 0 0 1, limit lower=-1.7453293 upper=1.7453293 effort=80 velocity=5
- added joint right_wrist_02: type revolute, parent L_Forearm_Upper_Drive, child KB-C-501X_Bayonet_Adapter_Hard_Stop_2, origin xyz=0.017349999973205105 -0.1055 0.018 rpy=1.5707963000000003 -1.5707963 0.0, axis 0 0 -1, limit lower=-1.7453293 upper=1.7453293 effort=80 velocity=5
- joint floating_base: child body1-part -> KB-B-102B_TORSO_BOTTOM

Commit message: Fix Robot URDF

File: public/cad/gpr-20241204.urdf (robot description, URDF)
Before this commit: robot robot_assy, 22 links, 21 joints
Links:
- removed link RS03
- removed link RS03_2
- added link RS03_5, mass 1.861434012; collision mesh filename=meshes/RS03_5_collision.stl; visual mesh filename=meshes/RS03_5.stl
- added link RS03_6, mass 1.86146043; collision mesh filename=meshes/RS03_6_collision.stl; visual mesh filename=meshes/RS03_6.stl
- added link imu, mass 0.0057; visual mesh filename=meshes/imu.stl
- link KB-B-102B_TORSO_BOTTOM: geometry collision mesh filename=meshes/KB-B-102B_TORSO_BOTTOM_collision.stl; visual mesh filename=meshes/KB-B-102B_TORSO_BOTTOM.stl
- link KB-C-101L_ShldYokeROLL: geometry visual mesh filename=meshes/KB-C-101L_ShldYokeROLL.stl
- link KB-C-101R_R_Shoulder_Drive: geometry visual mesh filename=meshes/KB-C-101R_R_Shoulder_Drive.stl
- link KB-C-501X_Bayonet_Adapter_Hard_Stop: geometry collision mesh filename=meshes/KB-C-501X_Bayonet_Adapter_Hard_Stop.convex.stl; visual mesh filename=meshes/KB-C-501X_Bayonet_Adapter_Hard_Stop.stl
- link KB-C-501X_Bayonet_Adapter_Hard_Stop_2: geometry collision mesh filename=meshes/KB-C-501X_Bayonet_Adapter_Hard_Stop_2.convex.stl; visual mesh filename=meshes/KB-C-501X_Bayonet_Adapter_Hard_Stop_2.stl
- link KB-D-102L_L_Hip_Yoke_Drive: geometry visual mesh filename=meshes/KB-D-102L_L_Hip_Yoke_Drive.stl
- link KB-D-102R_R_Hip_Yoke_Drive: geometry visual mesh filename=meshes/KB-D-102R_R_Hip_Yoke_Drive.stl
- link KB-D-301L_L_Femur_Lower_Drive: geometry collision mesh filename=meshes/KB-D-301L_L_Femur_Lower_Drive_collision.stl; visual mesh filename=meshes/KB-D-301L_L_Femur_Lower_Drive.stl
- link KB-D-301R_R_Femur_Lower_Drive: geometry collision mesh filename=meshes/KB-D-301R_R_Femur_Lower_Drive_collision.stl; visual mesh filename=meshes/KB-D-301R_R_Femur_Lower_Drive.stl
- link KB-D-401L_L_Shin_Drive: geometry collision mesh filename=meshes/KB-D-401L_L_Shin_Drive_collision.stl; visual mesh filename=meshes/KB-D-401L_L_Shin_Drive.stl
- link KB-D-401R_R_Shin_Drive: geometry collision mesh filename=meshes/KB-D-401R_R_Shin_Drive_collision.stl; visual mesh filename=meshes/KB-D-401R_R_Shin_Drive.stl
- link KB-D-501L_L_LEG-FOOT: geometry collision mesh filename=meshes/KB-D-501L_L_LEG-FOOT.convex.stl; visual mesh filename=meshes/KB-D-501L_L_LEG-FOOT.stl
- link KB-D-501R_R_LEG-FOOT: geometry collision mesh filename=meshes/KB-D-501R_R_LEG-FOOT.convex.stl; visual mesh filename=meshes/KB-D-501R_R_LEG-FOOT.stl
- link L_Bicep_Lower_Drive: geometry collision mesh filename=meshes/L_Bicep_Lower_Drive_collision.stl; visual mesh filename=meshes/L_Bicep_Lower_Drive.stl
- link L_Forearm_Upper_Drive: geometry collision mesh filename=meshes/L_Forearm_Upper_Drive_collision.stl; visual mesh filename=meshes/L_Forearm_Upper_Drive.stl
- link RS03_3: mass 1.861434012 -> 2.5903163030000003; geometry collision mesh filename=meshes/RS03_3_collision.stl; visual mesh filename=meshes/RS03_3.stl
- link RS03_4: mass 1.86146043 -> 2.590428564; geometry collision mesh filename=meshes/RS03_4_collision.stl; visual mesh filename=meshes/RS03_4.stl
- link R_Bicep_Lower_Drive: geometry collision mesh filename=meshes/R_Bicep_Lower_Drive_collision.stl; visual mesh filename=meshes/R_Bicep_Lower_Drive.stl
- link R_Forearm_Upper_Structural: geometry collision mesh filename=meshes/R_Forearm_Upper_Structural_collision.stl; visual mesh filename=meshes/R_Forearm_Upper_Structural.stl
Joints:
- removed joint left_hip_yaw_03
- removed joint right_hip_yaw_03
- added joint imu_link: type fixed, parent KB-B-102B_TORSO_BOTTOM, child imu, origin xyz=-4.488159466925432e-05 0.009977114961696199 0.40030576959807607 rpy=-3.136765140794895 -2.6794895413573272e-08 -9.999999983634211e-08
- added joint left_hip_yaw_: type revolute, parent RS03_4, child KB-D-301L_L_Femur_Lower_Drive, origin xyz=0.0 -0.14275000000000002 -0.0297999999732051 rpy=1.5707963 0.0 0.0, axis 0 0 -1, limit lower=-1.5707963 upper=1.9198622 effort=17 velocity=360
- added joint right_hip_yaw_02: type revolute, parent RS03_3, child KB-D-301R_R_Femur_Lower_Drive, origin xyz=0.0 -0.14275 -0.0297999999732051 rpy=1.5707963 0.0 0.0, axis 0 0 -1, limit lower=-1.5707963 upper=1.9198622 effort=17 velocity=12.566
- joint floating_base: origin xyz=0 0 0 rpy=0 0 0 -> xyz=0.0 0.0 -0.001 rpy=0.00 0.00 3.14; type fixed -> floating
- joint left_ankle_02: limit lower=-0.29670597 upper=0.78539816 effort=80 velocity=5 -> lower=-0.29670597 upper=0.78539816 effort=17 velocity=12.566; origin xyz=-0.0313 0.2925 0.005 rpy=3.1415927 0 0 -> xyz=-0.0313 0.2924999999535898 0.005999999999999999 rpy=3.1415927 0 0
- joint left_elbow_02: limit lower=0 upper=2.5307274 effort=80 velocity=5 -> lower=0 upper=2.5307274 effort=17 velocity=12.566; origin xyz=0.01749999579319584 -0.010000000468910617 -0.13699999843121974 rpy=-1.5707963646886025 2.6794895413573272e-08 1.5707962999999985 -> xyz=0.01849999579319584 -0.010000000495705515 -0.13699999839332602 rpy=-1.5707963646886025 2.6794895413573272e-08 1.5707962999999985
- joint left_hip_pitch_04: limit lower=-1.5707963 upper=1.9198622 effort=80 velocity=5 -> lower=-1.5707963 upper=1.9198622 effort=120 velocity=6.283; origin xyz=-0.047048021999999995 -0.000737257000000005 -0.07299347924500096 rpy=-1.5707963 2.6794896523796297e-08 -1.5707963267948961 -> xyz=-0.048048021999999996 -0.0007372570000000047 -0.07299347927179586 rpy=-1.5707963 2.6794896523796297e-08 -1.5707963267948961
- joint left_hip_roll_03: child RS03_2 -> RS03_4; limit lower=-0.20943951 upper=2.6179939 effort=80 velocity=5 -> lower=-0.20943951 upper=2.6179939 effort=60 velocity=6.283; origin xyz=-0.02925 0.03 -0.071 rpy=3.1415927 1.5707963 0 -> xyz=-0.028250000000000004 0.029999999953589793 -0.0709999999732051 rpy=3.1415927 1.5707963 0
- joint left_knee_04: limit lower=-2.6703538 upper=0 effort=80 velocity=5 -> lower=-2.6703538 upper=0 effort=120 velocity=6.283; origin xyz=0.019600006618339327 0.02099999745046268 -0.2119999988276073 rpy=-1.5707963646886016 2.6794893859261038e-08 1.5707962535897926 -> xyz=0.02059999707935614 -0.02099999737725783 0.21199999817878992 rpy=1.5707962889011908 -2.6794893859261038e-08 -1.5707962535897921
- joint left_shoulder_pitch_03: limit lower=-1.9198622 upper=3.4906585 effort=80 velocity=5 -> lower=-1.9198622 upper=3.4906585 effort=60 velocity=6.283; origin xyz=0.1249499752752948 -0.000737260654998772 0.3375065237953634 rpy=1.570796364688602 -7.320510020392135e-08 -1.5707964000000025 -> xyz=0.1259499752752948 -0.0007372607282038752 0.3375065238332571 rpy=1.570796364688602 -7.320510020392135e-08 -1.5707964000000025
- joint left_shoulder_roll_03: child RS03_3 -> RS03_5; limit lower=-1.4835299 upper=0.48869219 effort=80 velocity=5 -> lower=-1.4835299 upper=0.48869219 effort=60 velocity=6.283; origin xyz=-0.02525 0 -0.075 rpy=0 -1.5707963 0 -> xyz=-0.02425 0.0 -0.0750000000267949 rpy=0 -1.5707963 0
- joint left_shoulder_yaw_02: limit lower=-1.7453293 upper=1.7453293 effort=80 velocity=5 -> lower=-1.7453293 upper=1.7453293 effort=17 velocity=12.566; origin xyz=-0.013 -0.14099999871210736 -0.03025020663762125 rpy=-1.570796207179587 0.0 0.0 -> xyz=-0.013 -0.14199999871210736 -0.03025020675723656 rpy=-1.570796207179587 0.0 0.0; parent RS03_3 -> RS03_5
- joint left_wrist_02: limit lower=-1.7453293 upper=1.7453293 effort=80 velocity=5 -> lower=-1.7453293 upper=1.7453293 effort=17 velocity=12.566; origin xyz=0.017350000026794897 0.1055 0.018 rpy=1.5707963999999996 1.5707963000000005 0.0 -> xyz=0.0173500001 0.1065 0.018000000000000002 rpy=1.5707963999999996 1.5707963000000005 0.0
- joint right_ankle_02: limit lower=-0.29670597 upper=0.78539816 effort=80 velocity=5 -> lower=-0.29670597 upper=0.78539816 effort=17 velocity=12.566; origin xyz=-0.0313 -0.2925 0.005 rpy=0 0 0 -> xyz=-0.0313 -0.2925 0.006 rpy=0 0 0
- joint right_elbow_02: limit lower=-2.5307274 upper=0 effort=80 velocity=5 -> lower=-2.5307274 upper=0 effort=17 velocity=12.566; origin xyz=-0.017499996329093773 -0.009999999531089408 -0.1370000008185232 rpy=1.5707962889011908 2.6794895413573272e-08 1.5707962999999994 -> xyz=-0.01849999632909377 -0.009999999504294511 -0.13700000085641692 rpy=1.5707962889011908 2.6794895413573272e-08 1.5707962999999994
- joint right_hip_pitch_04: limit lower=-1.9198622 upper=1.5707963 effort=80 velocity=5 -> lower=-1.9198622 upper=1.5707963 effort=120 velocity=6.283; origin xyz=0.04704799199999996 -0.0007372588099980745 -0.07299347715499904 rpy=1.570796353589793 2.6794898300153136e-08 -1.570796373205102 -> xyz=0.04804799199999996 -0.0007372588564082805 -0.07299347712820414 rpy=1.570796353589793 2.6794898300153136e-08 -1.570796373205102
- joint right_hip_roll_03: child RS03 -> RS03_3; limit lower=-2.6179939 upper=0.20943951 effort=80 velocity=5 -> lower=-2.6179939 upper=0.20943951 effort=60 velocity=6.283; origin xyz=-0.02925 -0.03 -0.071 rpy=0 -1.5707963 0 -> xyz=-0.02825 -0.03 -0.0710000000267949 rpy=0 -1.5707963 0
- joint right_knee_04: limit lower=0 upper=2.6703538 effort=80 velocity=5 -> lower=0 upper=2.6703538 effort=120 velocity=6.283; origin xyz=-0.019600005492953775 0.02099999892954119 -0.21199999882760728 rpy=1.5707963646886023 -2.6794896967885506e-08 1.5707963464102066 -> xyz=-0.02059999595397059 -0.020999998909925658 0.21199999817878992 rpy=-1.570796288901191 2.6794897411974716e-08 -1.5707963464102055
- joint right_shoulder_pitch_03: limit lower=-1.9198622 upper=3.4906585 effort=80 velocity=5 -> lower=-1.9198622 upper=3.4906585 effort=60 velocity=6.283; origin xyz=-0.12495002472470498 -0.0007372555262804718 0.33750651980463664 rpy=-1.5707963182783953 2.6794895635617877e-08 1.5707962999999996 -> xyz=-0.12595002472470498 -0.0007372554994855747 0.33750651981315316 rpy=-1.5707963182783953 2.6794895635617877e-08 1.5707962999999996
- joint right_shoulder_roll_03: child RS03_4 -> RS03_6; limit lower=-0.48869219 upper=1.4835299 effort=80 velocity=5 -> lower=-0.48869219 upper=1.4835299 effort=60 velocity=6.283; origin xyz=0.02525 0 0.075 rpy=3.1415927 -1.5707963 0 -> xyz=0.024250000000000004 -4.6410206666284833e-11 0.0750000000267949 rpy=3.1415927 -1.5707963 0
- joint right_shoulder_yaw_02: limit lower=-1.7453293 upper=1.7453293 effort=80 velocity=5 -> lower=-1.7453293 upper=1.7453293 effort=17 velocity=12.566; origin xyz=0.012999999999999998 -0.14099999871210692 -0.03025021299389611 rpy=-1.5707962143591734 0.0 0.0 -> xyz=0.012999999999999998 -0.14199999871210692 -0.030250213106331834 rpy=-1.5707962143591734 0.0 0.0; parent RS03_4 -> RS03_6
- joint right_wrist_02: limit lower=-1.7453293 upper=1.7453293 effort=80 velocity=5 -> lower=-1.7453293 upper=1.7453293 effort=17 velocity=12.566; origin xyz=0.017349999973205105 -0.1055 0.018 rpy=1.5707963000000003 -1.5707963 0.0 -> xyz=0.01734999994641021 -0.1065 0.018 rpy=1.5707963000000003 -1.5707963 0.0
